File: PD-AuxPower-Card-PCB/Power_Stage.kicad_sch (KiCad schematic)
At the start: 31 parts, among them J4 2.54mm terminal, Q1 FDMC86520L, T1 ER 9.5, U8 LTV-217, U9 TLV431BFTA

Commit message: FEAT: Revolution PCB to ver 1.0. Change COMP1+ to 3v3 current sense, COMP2+ to 12V current sense and 12V LED to GPIO7 output. Modify PCB layout.
Parts:
- removed C24: 1n/500V, Capacitor_SMD:C_1210_3225Metric, symbol Device:C_Small
- added C3: 2200p/500V, Capacitor_SMD:C_1206_3216Metric, symbol Device:C_Small
- R26: value 8.2k -> 0
- R3: value 0 -> 8.2k
- T1: footprint User:Transformer_ER9.5_11.6mmx8.2mm -> Johnson's:Transformer_ER9.5_11.6mmx8.2mm
Connections:
- net GND: now also C3.1
- net GND1: now also C3.2
Other:
- company: (none) -> Habonroof Playground
- title: (none) -> 3.3/5V Flyback converter
Changed lines of the file:
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@@
 (kicad_sch (version 20230121) (generator eeschema)
   (paper "A4")
+  (title_block
+    (title "3.3/5V Flyback converter")
+    (date "2023-11-26")
+    (rev "Rev 1.0")
+    (company "Habonroof Playground")
+  )
   (junction (at 146.05 109.22) (diameter 0) (color 0 0 0 0)
   )
@@
     (stroke (width 0) (type default))
   )
+  (wire (pts (xy 144.78 151.765) (xy 149.225 151.765))
+    (stroke (width 0) (type default))
+  )
   (wire (pts (xy 159.385 67.945) (xy 160.655 67.945))
     (stroke (width 0) (type default))
@@
     (stroke (width 0) (type default))
   )
-  (wire (pts (xy 154.305 131.445) (xy 158.115 131.445))
-    (stroke (width 0) (type default))
-  )
   (wire (pts (xy 192.405 85.09) (xy 217.17 85.09))
     (stroke (width 0) (type default))
@@
     (stroke (width 0) (type default))
   )
-  (wire (pts (xy 149.225 131.445) (xy 145.415 131.445))
-    (stroke (width 0) (type default))
-  )
   (wire (pts (xy 88.265 118.745) (xy 95.885 118.745))
     (stroke (width 0) (type default))
@@
     (stroke (width 0) (type default))
   )
+  (wire (pts (xy 133.985 151.765) (xy 139.7 151.765))
+    (stroke (width 0) (type default))
+  )
   (wire (pts (xy 178.435 75.565) (xy 178.435 78.105))
     (stroke (width 0) (type default))
@@
     (stroke (width 0) (type default))
   )
-  (wire (pts (xy 158.115 131.445) (xy 158.115 133.985))
-    (stroke (width 0) (type default))
-  )
   (wire (pts (xy 194.945 121.92) (xy 217.17 121.92))
     (stroke (width 0) (type default))
@@
     (stroke (width 0) (type default))
   )
-  (wire (pts (xy 145.415 131.445) (xy 145.415 133.985))
-    (stroke (width 0) (type default))
-  )
   (wire (pts (xy 200.025 67.945) (xy 210.82 67.945))
     (stroke (width 0) (type default))
@@
     (stroke (width 0) (type default))
   )
+  (wire (pts (xy 149.225 151.765) (xy 149.225 154.305))
+    (stroke (width 0) (type default))
+  )
   (wire (pts (xy 88.265 62.23) (xy 88.265 55.88))
     (stroke (width 0) (type default))
@@
   )
   (wire (pts (xy 111.125 84.455) (xy 111.125 86.995))
+    (stroke (width 0) (type default))
+  )
+  (wire (pts (xy 133.985 154.305) (xy 133.985 151.765))
     (stroke (width 0) (type default))
   )
@@
     (effects (font (size 1.27 1.27)) (justify left bottom))
   )
-  (text "1:1:3" (at 146.685 57.785 0)
+  (text "1:1:3" (at 146.685 57.15 0)
     (effects (font (size 1.27 1.27)) (justify left bottom))
   )
@@
   (hierarchical_label "Cur_FB_5V" (shape output) (at 88.265 118.745 180) (fields_autoplaced)
     (effects (font (size 1.27 1.27)) (justify right))
-  )
-  (symbol (lib_id "power:GND") (at 145.415 133.985 0) (unit 1)
-    (in_bom yes) (on_board yes) (dnp no) (fields_autoplaced)
-    (property "Reference" "#PWR08" (at 145.415 140.335 0)
-      (effects (font (size 1.27 1.27)) hide)
-    )
-    (property "Value" "GND" (at 145.415 139.065 0)
-      (effects (font (size 1.27 1.27)))
-    )
-    (property "Footprint" "" (at 145.415 133.985 0)
-      (effects (font (size 1.27 1.27)) hide)
-    )
-    (property "Datasheet" "" (at 145.415 133.985 0)
-      (effects (font (size 1.27 1.27)) hide)
-    )
-    (pin "1")
-    (instances
-      (project "PD-AuxPower-Card"
-        (path "/48c5bc14-ccc3-44de-b526-838e3d53c0ee"
-          (reference "#PWR08") (unit 1)
-        )
-        (path "/48c5bc14-ccc3-44de-b526-838e3d53c0ee/40f113c1-6183-4863-b2ec-a4ca33698158"
-          (reference "#PWR068") (unit 1)
-        )
-      )
-    )
   )
   (symbol (lib_id "power:GND") (at 100.965 102.87 0) (unit 1)
@@
       (effects (font (size 1.27 1.27)) (justify right))
     )
-    (property "Value" "8.2k" (at 218.6686 95.8923 0)
+    (property "Value" "0" (at 218.6686 95.8923 0)
       (effects (font (size 1.27 1.27)) (justify right))
     )
@@
       (effects (font (size 1.27 1.27)) (justify right))
     )
-    (property "Value" "0" (at 218.6686 109.8623 0)
+    (property "Value" "8.2k" (at 218.6686 109.8623 0)
       (effects (font (size 1.27 1.27)) (justify right))
     )
@@
     )
   )
-  (symbol (lib_id "Device:C_Small") (at 151.765 131.445 90) (mirror x) (unit 1)
-    (in_bom yes) (on_board yes) (dnp no)
-    (property "Reference" "C24" (at 151.7713 136.017 90)
-      (effects (font (size 1.27 1.27)))
-    )
-    (property "Value" "1n/500V" (at 151.7713 134.096 90)
-      (effects (font (size 1.27 1.27)))
-    )
-    (property "Footprint" "Capacitor_SMD:C_1210_3225Metric" (at 151.765 131.445 0)
-      (effects (font (size 1.27 1.27)) hide)
-    )
-    (property "Datasheet" "~" (at 151.765 131.445 0)
-      (effects (font (size 1.27 1.27)) hide)
-    )
-    (pin "1")
-    (pin "2")
-    (instances
-      (project "PD-AuxPower-Card"
-        (path "/48c5bc14-ccc3-44de-b526-838e3d53c0ee/40f113c1-6183-4863-b2ec-a4ca33698158"
-          (reference "C24") (unit 1)
-        )
-      )
-    )
-  )
   (symbol (lib_id "Device:R_Small") (at 104.14 69.215 180) (unit 1)
     (in_bom yes) (on_board yes) (dnp no) (fields_autoplaced)
@@
     )
   )
+  (symbol (lib_id "Device:C_Small") (at 142.24 151.765 90) (unit 1)
+    (in_bom yes) (on_board yes) (dnp no) (fields_autoplaced)
+    (property "Reference" "C3" (at 142.2463 144.78 90)
+      (effects (font (size 1.27 1.27)))
+    )
+    (property "Value" "2200p/500V" (at 142.2463 147.32 90)
+      (effects (font (size 1.27 1.27)))
+    )
+    (property "Footprint" "Capacitor_SMD:C_1206_3216Metric" (at 142.24 151.765 0)
+      (effects (font (size 1.27 1.27)) hide)
+    )
+    (property "Datasheet" "~" (at 142.24 151.765 0)
+      (effects (font (size 1.27 1.27)) hide)
+    )
+    (pin "1")
+    (pin "2")
+    (instances
+      (project "PD-AuxPower-Card"
+        (path "/48c5bc14-ccc3-44de-b526-838e3d53c0ee/40f113c1-6183-4863-b2ec-a4ca33698158"
+          (reference "C3") (unit 1)
+        )
+      )
+    )
+  )
   (symbol (lib_id "Device:Transformer_1P_2S") (at 149.225 73.025 0) (mirror y) (unit 1)
     (in_bom yes) (on_board yes) (dnp no) (fields_autoplaced)
@@
       (effects (font (size 1.27 1.27)))
     )
-    (property "Footprint" "User:Transformer_ER9.5_11.6mmx8.2mm" (at 149.225 73.025 0)
+    (property "Footprint" "Johnson's:Transformer_ER9.5_11.6mmx8.2mm" (at 149.225 73.025 0)
       (effects (font (size 1.27 1.27)) hide)
     )
@@
     )
   )
+  (symbol (lib_id "power:GND1") (at 149.225 154.305 0) (unit 1)
+    (in_bom yes) (on_board yes) (dnp no) (fields_autoplaced)
+    (property "Reference" "#PWR014" (at 149.225 160.655 0)
+      (effects (font (size 1.27 1.27)) hide)
+    )
+    (property "Value" "GND1" (at 149.225 158.4405 0)
+      (effects (font (size 1.27 1.27)))
+    )
+    (property "Footprint" "" (at 149.225 154.305 0)
+      (effects (font (size 1.27 1.27)) hide)
+    )
+    (property "Datasheet" "" (at 149.225 154.305 0)
+      (effects (font (size 1.27 1.27)) hide)
+    )
+    (pin "1")
+    (instances
+      (project "PD-AuxPower-Card"
+        (path "/48c5bc14-ccc3-44de-b526-838e3d53c0ee/40f113c1-6183-4863-b2ec-a4ca33698158"
+          (reference "#PWR014") (unit 1)
+        )
+      )
+    )
+  )
   (symbol (lib_id "Device:R_Small") (at 104.14 61.595 180) (unit 1)
     (in_bom yes) (on_board yes) (dnp no) (fields_autoplaced)
@@
     )
   )
+  (symbol (lib_id "power:GND") (at 133.985 154.305 0) (unit 1)
+    (in_bom yes) (on_board yes) (dnp no)
+    (property "Reference" "#PWR08" (at 133.985 160.655 0)
+      (effects (font (size 1.27 1.27)) hide)
+    )
+    (property "Value" "GND" (at 133.985 158.75 0)
+      (effects (font (size 1.27 1.27)))
+    )
+    (property "Footprint" "" (at 133.985 154.305 0)
+      (effects (font (size 1.27 1.27)) hide)
+    )
+    (property "Datasheet" "" (at 133.985 154.305 0)
+      (effects (font (size 1.27 1.27)) hide)
+    )
+    (pin "1")
+    (instances
+      (project "PD-AuxPower-Card"
+        (path "/48c5bc14-ccc3-44de-b526-838e3d53c0ee"
+          (reference "#PWR08") (unit 1)
+        )
+        (path "/48c5bc14-ccc3-44de-b526-838e3d53c0ee/40f113c1-6183-4863-b2ec-a4ca33698158"
+          (reference "#PWR04") (unit 1)
+        )
+      )
+    )
+  )
   (symbol (lib_id "Device:C_Small") (at 111.125 65.405 0) (unit 1)
     (in_bom yes) (on_board yes) (dnp no) (fields_autoplaced)
@@
         )
       )
-    )
-  )
-  (symbol (lib_id "power:GND1") (at 158.115 133.985 0) (unit 1)
-    (in_bom yes) (on_board yes) (dnp no) (fields_autoplaced)
-    (property "Reference" "#PWR069" (at 158.115 140.335 0)
-      (effects (font (size 1.27 1.27)) hide)
-    )
-    (property "Value" "GND1" (at 158.115 138.1205 0)
-      (effects (font (size 1.27 1.27)))
-    )
-    (property "Footprint" "" (at 158.115 133.985 0)
-      (effects (font (size 1.27 1.27)) hide)
-    )
-    (property "Datasheet" "" (at 158.115 133.985 0)
-      (effects (font (size 1.27 1.27)) hide)
-    )
-    (pin "1")
-    (instances
-      (project "PD-AuxPower-Card"
-        (path "/48c5bc14-ccc3-44de-b526-838e3d53c0ee/40f113c1-6183-4863-b2ec-a4ca33698158"
-          (reference "#PWR069") (unit 1)
-        )
-      )

Commit message: FEAT: Add Matlab file (Octave capable) for calculation transformer parameter. Modify PCB schematic Redefine pinout, ISR and peripherial
Parts:
- R3: value 8.2k -> 6.8k
- R36: value 10k -> 6.8k
Changed lines of the file:
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@@
       (effects (font (size 1.27 1.27)) (justify right))
     )
-    (property "Value" "8.2k" (at 218.6686 109.8623 0)
+    (property "Value" "6.8k" (at 218.6686 109.8623 0)
       (effects (font (size 1.27 1.27)) (justify right))
     )
@@
       (effects (font (size 1.27 1.27)) (justify right))
     )
-    (property "Value" "10k" (at 219.71 129.54 0)
-      (effects (font (size 1.27 1.27)) (justify right))
-    )
+    (property "Value" "6.8k" (at 219.71 129.54 0)
+      (effects (font (size 1.27 1.27)) (justify right))
+    )
